File: KiCAD User Designs/Expansion_Bay_Template/Expansion_Bay.kicad_sch (KiCad schematic)
At the start: 5 parts, among them J1 FAN1, J3 FW_EBI, J5 FAN0

Commit message: Mess everything up
Parts:
- added J2: USB_C_Receptacle, symbol Connector:USB_C_Receptacle
- added R3, R5: 100k, symbol Device:R_Small_US
- added R4, R6: 1M, symbol Device:R_Small_US
- added SW1, SW2: U/D on flip, symbol Switch:SW_Push_DPDT
- added U1: ~, symbol pcieSlot:pcix8
Connections:
- net GND: now also J2.S1 (SHIELD), R4.2, R5.2
- net VADP_GPU: now reaches J3.PA1 (VADP_GPU), J3.PA2 (VADP_GPU), J3.PB1 (VADP_GPU), J3.PB2 (VADP_GPU), J3.PC1 (VADP_GPU), J3.PC2 (VADP_GPU)
- net 3V3_GND: now reaches J3.PA3 (3V3_GND), J3.PB3 (3V3_GND), J3.PE3 (3V3_GND)
- net 3V3_ALW: now reaches J3.PA4 (3V3_ALW), J3.PA5 (3V3_ALW), J3.PB4 (3V3_ALW), J3.PB5 (3V3_ALW)
- net VSYS_GND: now reaches J3.PA6 (VSYS_GND), J3.PB6 (VSYS_GND), J3.PC6 (VSYS_GND), J3.PD6 (VSYS_GND), J3.PE6 (VSYS_GND), J3.PF6 (VSYS_GND), J3.PG6 (VSYS_GND), J3.PH6 (VSYS_GND), J3.PH7 (VSYS_GND), J3.PH8 (VSYS_GND), J3.PJ7 (VSYS_GND), J3.PJ8 (VSYS_GND)
- net VSYS_GPU: now reaches J3.PA7 (VSYS_GPU), J3.PA8 (VSYS_GPU), J3.PB7 (VSYS_GPU), J3.PB8 (VSYS_GPU), J3.PC7 (VSYS_GPU), J3.PC8 (VSYS_GPU), J3.PD7 (VSYS_GPU), J3.PD8 (VSYS_GPU), J3.PE7 (VSYS_GPU), J3.PE8 (VSYS_GPU), J3.PF7 (VSYS_GPU), J3.PF8 (VSYS_GPU), J3.PG7 (VSYS_GPU), J3.PG8 (VSYS_GPU)
- net VADP_GND: now reaches J3.PD1 (VADP_GND), J3.PD2 (VADP_GND), J3.PE1 (VADP_GND), J3.PE2 (VADP_GND), J3.PF1 (VADP_GND)
- net USB_gnd: now reaches J3.PH3 (USB_GND), J3.PL3 (USB_GND)
- net USB_gnd: now also J2.A1 (GND), J2.A12 (GND), J2.B1 (GND), J2.B12 (GND)
- net USB+: now reaches J3.PJ3 (USB+)
- net USB+: now also J2.A6 (D+), J2.B6 (D+)
- net USB-: now reaches J3.PK3 (USB-)
- net USB-: now also J2.A7 (D-), J2.B7 (D-)
- net MI_SO_p6: now reaches J3.SA1 (PEX_RX6P)
- net MI_SO_p6: now also U1.B43 (HSIp6)
- net MI_SO_p4: now reaches J3.SA3 (PEX_RX4P)
- net MI_SO_p4: now also U1.B35 (HSIp4)
- net ReqCLK: now reaches J3.SA4 (PEX_CLK_REQ)
- net ReqCLK: now also U1.A12 (CLKREQ#)
- net PexRST: now reaches J3.SA5 (PEX_RST)
- net PexRST: now also U1.B11 (PERST#)
- net MI_SO_n3: now reaches J3.SA6 (PEX_RX3N)
- net MI_SO_n3: now also U1.B29 (HSIp3)
- net DP_HPD: now reaches J3.SA7 (DP_A_HPD)
- net MI_SO_n1: now reaches J3.SA8 (PEX_RX1N)
- net MI_SO_n1: now also U1.B21 (HSIp1)
- net MI_SO_n6: now reaches J3.SB1 (PEX_RX6N)
- net MI_SO_n6: now also U1.B44 (HSIn6)
- net PexGND: now reaches J3.SB2 (PEX_GND), J3.SB7 (PEX_GND), J3.SC1 (PEX_GND), J3.SC3 (PEX_GND), J3.SC6 (PEX_GND), J3.SC8 (PEX_GND), J3.SE2 (PEX_GND), J3.SE7 (PEX_GND), J3.SF1 (PEX_GND), J3.SF3 (PEX_GND), J3.SF6 (PEX_GND), J3.SF8 (PEX_GND), J3.SH2 (PEX_GND), J3.SH7 (PEX_GND), J3.SJ1 (PEX_GND), J3.SJ3 (PEX_GND), J3.SJ6 (PEX_GND), J3.SJ8 (PEX_GND)
- net PexGND: now also U1.A04 (GND), U1.A07 (GND), U1.A13 (GND), U1.A16 (GND), U1.A18 (GND), U1.A21 (GND), U1.A22 (GND), U1.A25 (GND), U1.A26 (GND), U1.A29 (GND), U1.A32 (GND), U1.A35 (GND), U1.A36 (GND), U1.A39 (GND), U1.A40 (GND), U1.A43 (GND), U1.A44 (GND), U1.A47 (GND), U1.A49 (GND), U1.B04 (GND), U1.B12 (GND), U1.B15 (GND), U1.B18 (GND), U1.B20 (GND), U1.B23 (GND), U1.B24 (GND), U1.B27 (GND), U1.B28 (GND), U1.B31 (GND), U1.B34 (GND), U1.B37 (GND), U1.B38 (GND), U1.B41 (GND), U1.B42 (GND), U1.B45 (GND), U1.B46 (GND), U1.B49 (GND)
- net MI_SO_n4: now reaches J3.SB3 (PEX_RX4N)
- net MI_SO_n4: now also U1.B36 (HSIn4)
- net MI_SO_p3: now reaches J3.SB6 (PEX_RX3P)
- net MI_SO_p3: now also U1.B30 (HSIn3)
- net MI_SO_p1: now reaches J3.SB8 (PEX_RX1P)
- net MI_SO_p1: now also U1.B22 (HSIn1)
- net RefCLKp: now reaches J3.SC2 (PEX_REFCLK_P)
- net RefCLKp: now also U1.B13 (REFCLK+)
- net DP_L1n: now reaches J3.SC7 (DP_A_L1N)
- net DP_L1n: now also J2.B3 (TX2-)
- net MI_SO_n7: now reaches J3.SD1 (PEX_RX7N)
- net MI_SO_n7: now also U1.B47 (HSIp7)
- net RefCLKn: now reaches J3.SD2 (PEX_REFCLK_N)
- net RefCLKn: now also U1.B14 (REFCLK-)
- net MI_SO_p5: now reaches J3.SD3 (PEX_RX5P)
- net MI_SO_p5: now also U1.B40 (HSIn5)
- net MI_SO_n2: now reaches J3.SD6 (PEX_RX2N)
- net MI_SO_n2: now also U1.B26 (HSIn2)
- net DP_L1p: now reaches J3.SD7 (DP_A_L1P)
- net DP_L1p: now also J2.B2 (TX2+)
- net MI_SO_n0: now reaches J3.SD8 (PEX_RX0N)
- net MI_SO_n0: now also U1.B17 (HSIn0)
- net MI_SO_p7: now reaches J3.SE1 (PEX_RX7P)
- net MI_SO_p7: now also U1.B48 (HSIn7)
- net MI_SO_n5: now reaches J3.SE3 (PEX_RX5N)
- net MI_SO_n5: now also U1.B39 (HSIp5)
- net MI_SO_p2: now reaches J3.SE6 (PEX_RX2P)
- net MI_SO_p2: now also U1.B25 (HSIp2)
- net MI_SO_p0: now reaches J3.SE8 (PEX_RX0P)
- net MI_SO_p0: now also U1.B16 (HSIp0)
- net DP_L3n: now reaches J3.SF2 (DP_A_L3N)
- net DP_L3n: now also J2.B10 (RX1-)
- net DP_L0n: now reaches J3.SF7 (DP_A_L0N)
- net DP_L0n: now also J2.A10 (RX2-)
- net DP_L3p: now reaches J3.SG2 (DP_A_L3P)
- net DP_L3p: now also J2.B11 (RX1+)
- net DP_L0p: now reaches J3.SG7 (DP_A_L0P)
- net DP_L0p: now also J2.A11 (RX2+)
- net DP_L2n: now reaches J3.SJ2 (DP_A_L2N)
- net DP_L2n: now also J2.A3 (TX1-)
- net DP_AUXn: now reaches J3.SJ7 (DP_A_AUXN)
- net DP_AUXn: now also SW1.1 (A), SW1.6 (C), SW2.2 (B)
- net DP_L2p: now reaches J3.SK2 (DP_A_L2P)
- net DP_L2p: now also J2.A2 (TX1+)
- net DP_AUXp: now reaches J3.SK7 (DP_A_AUXP)
- net DP_AUXp: now also SW1.3 (C), SW1.4 (A), SW2.5 (B)
- new net: R6.1, SW2.4 (A)
- new net: J2.A4 (VBUS), J2.A9 (VBUS), J2.B4 (VBUS), J2.B9 (VBUS)
- new net: R4.1, SW2.1 (A)
- new net: R3.1, SW2.3 (C)
- new net: R5.1, SW2.6 (C)
- new net: U1.A01 (12V), U1.A02 (12V), U1.A03 (12V), U1.B02 (12V), U1.B03 (12V)
- new net: U1.A08 (3V3), U1.B09 (3V3), U1.B10 (3V3)
- new net: U1.A17 (PRSNT#2), U1.A31 (PRSNT#2), U1.A48 (PRSNT#2)
- new net 3v3: R3.2, R6.2
- new net MO_SI_n0: U1.A15 (HSOn0)
- new net MO_SI_n1: U1.A20 (HSOn1)
- new net MO_SI_n2: U1.A24 (HSOn2)
- new net MO_SI_n3: U1.A28 (HSOn3)
- new net MO_SI_n4: U1.A34 (HSOn4)
- new net MO_SI_n5: U1.A38 (HSOn5)
- new net MO_SI_n6: U1.A42 (HSOn6)
- new net MO_SI_n7: U1.A46 (HSOn7)
- new net MO_SI_p0: U1.A14 (HSOp0)
- new net MO_SI_p1: U1.A19 (HSOp1)
- new net MO_SI_p2: U1.A23 (HSOp2)
- new net MO_SI_p3: U1.A27 (HSOp3)
- new net MO_SI_p4: U1.A33 (HSOp4)
- new net MO_SI_p5: U1.A37 (HSOp5)
- new net MO_SI_p6: U1.A41 (HSOp6)
- new net MO_SI_p7: U1.A45 (HSOp7)
- new net SBU1: J2.A8 (SBU1), SW1.2 (B)
- new net SBU2: J2.B8 (SBU2), SW1.5 (B)
Other:
- note added: "ALL OF THIS MIGHT BE FLIPPED A/B!"
- note added: "Switch changes if UFD_D or DFD_D (UFP_D def)"
- note added: "flipped/unflipped, signal for PD"
- moved on the sheet: J1, J5
